File: rocketpanda_hw/rockpanda_v1_hardware/rocketpanda_v1.brd (EAGLE design)
At the start: 86.4 x 54.6 mm, 40 parts, among them J2 JTAG, Q1 MC-306, U1 FTS31XS-U

Commit message: updated hardware files!
Connections:
- removed net P006: J1.9
- removed net P008: J1.13
- removed net RESET: C7.2, D1.A, R5.1
- net DTR: now also U1.1; no longer U1.14
- net NRST: now also C7.2, D1.A, R5.1
- net RX: now also J1.13
- net SWCLK: no longer J2.4, U$1.P36
- net SWDCLK: now also J2.4, U$1.P36
- net TX: now also J1.9
Routing:
- net TX: track 77.6 -> 214.0 mm, vias 4 -> 3
- net SWCLK: track 104.0 -> 0.00 mm, vias 1 -> 0
- net SWDCLK: track 0.00 -> 90.2 mm
- net RX: track 61.8 -> 128.8 mm, vias 3 -> 5
- net GND: track 369.7 -> 317.7 mm, vias 7 -> 12
- net NRST: track 63.7 -> 100.1 mm, vias 2 -> 5
- net 3.3V: track 180.8 -> 156.3 mm, vias 1 -> 5
- net N$4: track 32.0 -> 8.14 mm
- net DTR: track 6.73 -> 29.6 mm
- net P012: track 26.7 -> 47.5 mm, vias 2 -> 4
- net P018: track 91.6 -> 72.6 mm, vias 5 -> 3
- net P009: track 32.8 -> 48.4 mm, vias 0 -> 4
- net P007: track 65.2 -> 80.0 mm
- net N$3: track 25.6 -> 12.0 mm
- net P019: track 102.7 -> 90.8 mm, vias 2 -> 1
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