File: rocketpanda_hw/rockpanda_v1_hardware/rocketpanda_v1.sch (EAGLE design)
At the start: 40 parts, among them J2 JTAG, J5 USB_MINI-B_SMT, Q1 MC-306, U1 FTS31XS-U, X1 B4B-PH-SM4-TB

Commit message: updated hardware files!
Connections:
- removed net P006: J1.9
- removed net P008: J1.13
- removed net RESET: C7.2, D1.A, R5.1
- net DTR: now also U1.!DTR; no longer U1.!RESET
- net NRST: now also C7.2, D1.A, R5.1
- net RX: now also J1.13
- net SWCLK: no longer J2.SWDCLK/TCK, U$1.P36-SWDCLK
- net SWDCLK: now also J2.SWDCLK/TCK, U$1.P36-SWDCLK
- net TX: now also J1.9
